Commit message: Add files via upload

File: urdf/smr100l_description.urdf (robot description, URDF)
Before this commit: robot smr100l_description, 18 links, 17 joints
Links:
- link base_link: mass 28.1550787286733 -> 28.155
- link caster_front_left_arm_link: mass 0.0620885720640709 -> 0.062089
- link caster_front_left_wheel_link: mass 0.352528491588121 -> 0.35253
- link caster_front_right_arm_link: mass 0.0620885720820533 -> 0.062089
- link caster_front_right_wheel_link: mass 0.352528489887363 -> 0.35253
- link caster_rear_left_arm_link: mass 0.062088572117153 -> 0.062089
- link caster_rear_left_wheel_link: mass 0.35252848990743 -> 0.35253
- link caster_rear_right_arm_link: mass 0.0620885721317263 -> 0.062089
- link caster_rear_right_wheel_link: mass 0.35252848990743 -> 0.35253
- link depthcam_link: mass 0.0364722975832015 -> 0.036472
- link imu_link: mass 0.000911356888660498 -> 0.00091136
- link lidar_front_right_link: mass 0.0481184286647859 -> 0.048118
- link lidar_rear_left_link: mass 0.0481184302326393 -> 0.048118
- link lifter_link: mass 28.8633842413996 -> 28.863
- link swing_arm_left_link: mass 9.18443575420952 -> 9.1844
- link swing_arm_right_link: mass 9.18423950420952 -> 9.1842
- link wheel_left_link: mass 4.95544635923129 -> 4.9554
- link wheel_right_link: mass 4.95544635924954 -> 4.9554
Joints:
- joint lidar_rear_left_joint: origin xyz=-0.44 0.2335 0.23335 rpy=0 0 -3.1416 -> xyz=-0.439999999999994 0.233499999999734 0.233349999999999 rpy=0 0 -3.14159265358979
- joint swing_arm_left_joint: origin xyz=0.1625 0.1975 0.15 rpy=0 0 0 -> xyz=0.162499999999998 0.1975 0.15 rpy=0 0 0
- joint swing_arm_right_joint: origin xyz=0.1625 -0.1975 0.15 rpy=0 0 0 -> xyz=0.162499999999999 -0.1975 0.15 rpy=0 0 0

Commit message: Update smr100l_description.urdf

File: urdf/smr100l_description.urdf (robot description, URDF)
Before this commit: robot smr100l_description, 18 links, 17 joints
Links:
- link caster_front_left_wheel_link: geometry collision cylinder length=0.039 radius=0.0625; visual mesh filename=package://smr100l_description/meshes/caster_front_left_whee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
- link caster_front_right_wheel_link: geometry collision cylinder length=0.039 radius=0.0625; visual mesh filename=package://smr100l_description/meshes/caster_front_right_whe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
- link caster_rear_left_wheel_link: geometry collision cylinder length=0.039 radius=0.0625; visual mesh filename=package://smr100l_description/meshes/caster_rear_left_wheel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
- link caster_rear_right_wheel_link: geometry collision cylinder length=0.039 radius=0.0625; visual mesh filename=package://smr100l_description/meshes/caster_rear_right_whee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
